File: GRR_KNOB_BOARD.kicad_sch (KiCad schematic)
At the start: 2 parts, among them J1 Conn_01x02_Socket, U1 TCAN330

Commit message: CORRECTED_KNOB_BOARD_UPDATED
Parts:
- added C1, C4: 47uF, Capacitor_THT:C_Radial_D5.0mm_H5.0mm_P2.00mm, symbol Device:C_US
- added C2, C3: 0.1uF, Capacitor_SMD:C_0805_2012Metric_Pad1.18x1.45mm_HandSolder, symbol Device:C_US
- added J2: 5V (Vout), TerminalBlock_Phoenix:TerminalBlock_Phoenix_MKDS-1,5-2-5.08_1x02_P5.08mm_Horizontal, symbol Connector:Conn_01x02_Pin
- added U2: LM7805_TO220, Package_TO_SOT_THT:TO-220-3_Vertical, symbol Regulator_Linear:LM7805_TO220
- added U3: Teensy4.1, symbol teensy:Teensy4.1
- J1: value Conn_01x02_Socket -> 12V (Vin); footprint (none) -> TerminalBlock_Phoenix:TerminalBlock_Phoenix_MKDS-1,5-2-5.08_1x02_P5.08mm_Horizontal
Connections:
- net GNDREF: now reaches J1.1 (Pin_1)
- net GNDREF: now also U1.2 (GND), C1.2, C2.2, C3.2, C4.2, J2.1 (Pin_1), U2.2 (GND), U3.1 (GND)
- net at J1.2 (Pin_2): now also C1.1, C3.1, U2.1 (VI)
- net at U1.1 (TXD): now also U3.3 (1_TX1_CTX2_MISO1)
- net +3V3: now reaches U1.3 (VCC)
- net +3V3: now also U3.46 (3V3)
- net at U1.4 (RXD): now also U3.2 (0_RX1_CRX2_CS1)
- new net +5V: C2.1, C4.1, J2.2 (Pin_2), U2.3 (VO), U3.48 (VIN)
Other:
- moved on the sheet: U1
